File: schematic/broam.kicad_sch (KiCad schematic)
At the start: 17 parts, among them Q1 Q_Photo_NPN, U1 STC8G1K08A, U2 MCP73831-2-OT

Commit message: broam: rename z "swiecaca-kulka", plaska struktura repo, porzadki w schemacie
Rename projektu i plikow (swiecaca-kulka -> broam): schemat, biblioteka symboli,
netlista, PDF, raport ERC oraz identyfikatory wewnatrz KiCad (lib_id,
nazwa projektu, nickname biblioteki).

Dokumentacja:
- trigger = ciemnosc to wersja WDROZONA, wstrzas/wibracja = wariant OPCJONALNY
  (bylo: "rozwazany i odrzucony") - README + docs/architektura.md,
- netlista blokowa zastapiona stanem faktycznym z schematic/broam.net
  (16 netow, 47 node'ow, 17 komponentow, realne nazwy netow),
- poprawione liczniki: 19 symboli, 48 etykiet globalnych (nie "48 sieci"),
- opis pulapek KiCad sprawdzonych empirycznie.

Konfiguracja agenta:
- AGENTS.md: struktura plaska bez hardware/<projekt>/, sekcja
  "KiCad - zasady praktyczne",
- .opencode: agent Engineer, skille circuit-simulation i
  mechatronics-integration, komendy /nowy-projekt i /przeglad-schematu.

Schemat (KiCad):
- dodane schematic/broam.kicad_pro (wzorzec KiCad 10) + sym-lib-table
  i fp-lib-table projektu; tabele dzialaja tylko z plikiem projektu,
- fix footprintu U1: Package_SO:SOP-8_3.9x4.9mm_P1.27mm nie istnieje
  -> Package_SO:SOIC-8_3.9x4.9mm_P1.27mm,
- biblioteka przepuszczona przez kicad-cli sym upgrade (format KiCad 9 -> 10)
  i zsynchronizowana kopia symbolu w schemacie (Update Symbols from Library),
- ERC: 0 bledow, 90 -> 69 ostrzezen (67x endpoint_off_grid, 2x isolated_pin_label
  dla ISP_RX/ISP_TX),
- netlista, PDF i raport ERC wygenerowane ponownie przez kicad-cli.
Parts:
- U1: footprint Package_SO:SOP-8_3.9x4.9mm_P1.27mm -> Package_SO:SOIC-8_3.9x4.9mm_P1.27mm; symbol swiecaca-kulka:STC8G1K08A -> broam:STC8G1K08A
Changed lines of the file:
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@@
 	)
 	(symbol
-		(lib_id "swiecaca-kulka:STC8G1K08A")
+		(lib_id "broam:STC8G1K08A")
 		(at 150 90 0)
 		(unit 1)
@@
 			)
 		)
-		(property "Footprint" "Package_SO:SOP-8_3.9x4.9mm_P1.27mm"
+		(property "Footprint" "Package_SO:SOIC-8_3.9x4.9mm_P1.27mm"
 			(at 150 74.76 0)
 			(show_name no)
@@
 		)
 		(instances
-			(project "swiecaca-kulka"
+			(project "broam"
 				(path "/0a1b2c3d-4e5f-6071-8293-a4b5c6d7e8f9"
 					(reference "U1")
@@
 		)
 		(instances
-			(project "swiecaca-kulka"
+			(project "broam"
 				(path "/0a1b2c3d-4e5f-6071-8293-a4b5c6d7e8f9"
 					(reference "D1")
@@
 		)
 		(instances
-			(project "swiecaca-kulka"
+			(project "broam"
 				(path "/0a1b2c3d-4e5f-6071-8293-a4b5c6d7e8f9"
 					(reference "Q1")
@@
 		)
 		(instances
-			(project "swiecaca-kulka"
+			(project "broam"
 				(path "/0a1b2c3d-4e5f-6071-8293-a4b5c6d7e8f9"
 					(reference "BT1")
@@
 		)
 		(instances
-			(project "swiecaca-kulka"
+			(project "broam"
 				(path "/0a1b2c3d-4e5f-6071-8293-a4b5c6d7e8f9"
 					(reference "U2")
@@
 		)
 		(instances
-			(project "swiecaca-kulka"
+			(project "broam"
 				(path "/0a1b2c3d-4e5f-6071-8293-a4b5c6d7e8f9"
 					(reference "L1")
@@
 		)
 		(instances
-			(project "swiecaca-kulka"
+			(project "broam"
 				(path "/0a1b2c3d-4e5f-6071-8293-a4b5c6d7e8f9"
 					(reference "C1")
@@
 		)
 		(instances
-			(project "swiecaca-kulka"
+			(project "broam"
 				(path "/0a1b2c3d-4e5f-6071-8293-a4b5c6d7e8f9"
 					(reference "C5")
@@
 		)
 		(instances
-			(project "swiecaca-kulka"
+			(project "broam"
 				(path "/0a1b2c3d-4e5f-6071-8293-a4b5c6d7e8f9"
 					(reference "R4")
@@
 		)
 		(instances
-			(project "swiecaca-kulka"
+			(project "broam"
 				(path "/0a1b2c3d-4e5f-6071-8293-a4b5c6d7e8f9"
 					(reference "R1")
@@
 		)
 		(instances
-			(project "swiecaca-kulka"
+			(project "broam"
 				(path "/0a1b2c3d-4e5f-6071-8293-a4b5c6d7e8f9"
 					(reference "R2")
@@
 		)
 		(instances
-			(project "swiecaca-kulka"
+			(project "broam"
 				(path "/0a1b2c3d-4e5f-6071-8293-a4b5c6d7e8f9"
 					(reference "R3")
@@
 		)
 		(instances
-			(project "swiecaca-kulka"
+			(project "broam"
 				(path "/0a1b2c3d-4e5f-6071-8293-a4b5c6d7e8f9"
 					(reference "R5")
@@
 		)
 		(instances
-			(project "swiecaca-kulka"
+			(project "broam"
 				(path "/0a1b2c3d-4e5f-6071-8293-a4b5c6d7e8f9"
 					(reference "C2")
@@
 		)
 		(instances
-			(project "swiecaca-kulka"
+			(project "broam"
 				(path "/0a1b2c3d-4e5f-6071-8293-a4b5c6d7e8f9"
 					(reference "C3")
@@
 		)
 		(instances
-			(project "swiecaca-kulka"
+			(project "broam"
 				(path "/0a1b2c3d-4e5f-6071-8293-a4b5c6d7e8f9"
 					(reference "C4")
@@
 		)
 		(instances
-			(project "swiecaca-kulka"
+			(project "broam"
 				(path "/0a1b2c3d-4e5f-6071-8293-a4b5c6d7e8f9"
 					(reference "D2")
@@
 		)
 		(instances
-			(project "swiecaca-kulka"
+			(project "broam"
 				(path "/0a1b2c3d-4e5f-6071-8293-a4b5c6d7e8f9"
 					(reference "#FLG01")
@@
 		)
 		(instances
-			(project "swiecaca-kulka"
+			(project "broam"
 				(path "/0a1b2c3d-4e5f-6071-8293-a4b5c6d7e8f9"
 					(reference "#FLG02")
